Commit message: Change hip joints from revolute to fixed for improved stability

File: urdf/my_robot.urdf (robot description, URDF)
Before this commit: robot spec_based_quadruped, 17 links, 16 joints
Joints:
- joint FL_hip_joint: type revolute -> fixed
- joint FR_hip_joint: type revolute -> fixed
- joint RL_hip_joint: type revolute -> fixed
- joint RR_hip_joint: type revolute -> fixed

Commit message: Update gait control parameters and URDF specifications for improved stability and performance

File: urdf/my_robot.urdf (robot description, URDF)
Before this commit: robot spec_based_quadruped, 17 links, 16 joints
Links:
- link FL_hip_link: mass 0.1 -> 0.385
- link FL_shank_link: mass 0.075 -> 0.145
- link FL_thigh_link: mass 0.075 -> 0.105; geometry collision cylinder length=0.105 radius=0.02; visual cylinder length=0.105 radius=0.02
- link FR_hip_link: mass 0.1 -> 0.385
- link FR_shank_link: mass 0.075 -> 0.145
- link FR_thigh_link: mass 0.075 -> 0.105; geometry collision cylinder length=0.105 radius=0.02; visual cylinder length=0.105 radius=0.02
- link RL_hip_link: mass 0.1 -> 0.385
- link RL_shank_link: mass 0.075 -> 0.145
- link RL_thigh_link: mass 0.075 -> 0.105; geometry collision cylinder length=0.105 radius=0.02; visual cylinder length=0.105 radius=0.02
- link RR_hip_link: mass 0.1 -> 0.385
- link RR_shank_link: mass 0.075 -> 0.145
- link RR_thigh_link: mass 0.075 -> 0.105; geometry collision cylinder length=0.105 radius=0.02; visual cylinder length=0.105 radius=0.02
- link base_link: mass 5.0 -> 1.62; geometry collision box size=0.49 0.26 0.0925; visual box size=0.49 0.26 0.0925
Joints:
- joint FL_hip_joint: origin xyz=0.195 0.145 0 rpy=0 0 0 -> xyz=0.19875 0.1535 0 rpy=0 0 0
- joint FL_shank_joint: limit lower=-2.5 upper=0 effort=10 velocity=10 -> lower=-2.5 upper=0 effort=11 velocity=10; origin xyz=0 0 -0.145 rpy=0 0 0 -> xyz=0 0 -0.105 rpy=0 0 0
- joint FL_thigh_joint: limit lower=-1.5 upper=1.5 effort=10 velocity=10 -> lower=-1.5 upper=1.5 effort=11 velocity=10; origin xyz=0 0.025 0 rpy=0 0 0 -> xyz=0 0.0235 0 rpy=0 0 0
- joint FR_hip_joint: origin xyz=0.195 -0.145 0 rpy=0 0 0 -> xyz=0.19875 -0.1535 0 rpy=0 0 0
- joint FR_shank_joint: limit lower=-2.5 upper=0 effort=10 velocity=10 -> lower=-2.5 upper=0 effort=11 velocity=10; origin xyz=0 0 -0.145 rpy=0 0 0 -> xyz=0 0 -0.105 rpy=0 0 0
- joint FR_thigh_joint: limit lower=-1.5 upper=1.5 effort=10 velocity=10 -> lower=-1.5 upper=1.5 effort=11 velocity=10; origin xyz=0 -0.025 0 rpy=0 0 0 -> xyz=0 -0.0235 0 rpy=0 0 0
- joint RL_hip_joint: origin xyz=-0.195 0.145 0 rpy=0 0 0 -> xyz=-0.16 0.1535 0 rpy=0 0 0
- joint RL_shank_joint: limit lower=-2.5 upper=0 effort=10 velocity=10 -> lower=-2.5 upper=0 effort=11 velocity=10; origin xyz=0 0 -0.145 rpy=0 0 0 -> xyz=0 0 -0.105 rpy=0 0 0
- joint RL_thigh_joint: limit lower=-1.5 upper=1.5 effort=10 velocity=10 -> lower=-1.5 upper=1.5 effort=11 velocity=10; origin xyz=0 0.025 0 rpy=0 0 0 -> xyz=0 0.0235 0 rpy=0 0 0
- joint RR_hip_joint: origin xyz=-0.195 -0.145 0 rpy=0 0 0 -> xyz=-0.16 -0.1535 0 rpy=0 0 0
- joint RR_shank_joint: limit lower=-2.5 upper=0 effort=10 velocity=10 -> lower=-2.5 upper=0 effort=11 velocity=10; origin xyz=0 0 -0.145 rpy=0 0 0 -> xyz=0 0 -0.105 rpy=0 0 0
- joint RR_thigh_joint: limit lower=-1.5 upper=1.5 effort=10 velocity=10 -> lower=-1.5 upper=1.5 effort=11 velocity=10; origin xyz=0 -0.025 0 rpy=0 0 0 -> xyz=0 -0.0235 0 rpy=0 0 0
